File: PCB/SoftStartLamp/_autosave-SoftStartLamp.kicad_pcb (KiCad board)
At the start: 2 copper layers, 80 x 70 mm, 64 parts, among them J1 24V, J2 Fan, J3 Lamp, K1 G2R-1-E, K2 G2R-1-E, Q1 AO3401, Q2 8050, Q3 8050, Q4 8050, Q5 8050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

Commit message: new submission
Parts:
- Q2, Q3, Q4, Q5, Q6, Q7, Q9: value 8050 -> 2N5551
- Q8: value 8550 -> 2N5401
- R13: value 10K -> 4.7K
- R24, R25: value 820K -> 470K
- R6: value 10K -> 4.7k
